File: BM1368.kicad_sch (KiCad schematic)
At the start: 39 parts, among them U2 BM1368_mode1, U9 BM1368_mode1

Commit message: DRC Check
Parts:
- removed R49: 10k, Resistor_SMD:R_0805_2012Metric, symbol Device:R
Connections:
- net U9-VDD3_1: now reaches C67.2, C69.1, U9.28 (VDD1_1)
- net U9-VDD2_1: now reaches C66.2, C67.1, U9.29 (VDD2_1)
- net U9-VDD1_1: now reaches C63.2, C66.1, U9.30 (VDD3_1)
Changed lines of the file:
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@@
 	)
 	(junction
-		(at 254 55.88)
-		(diameter 0)
-		(color 0 0 0 0)
-	)
-	(junction
 		(at 78.74 36.83)
 		(diameter 0)
@@
 	)
 	(junction
+		(at 246.38 48.26)
+		(diameter 0)
+		(color 0 0 0 0)
+	)
+	(junction
 		(at 78.74 53.34)
 		(diameter 0)
@@
 	)
 	(junction
+		(at 257.81 50.8)
+		(diameter 0)
+		(color 0 0 0 0)
+	)
+	(junction
 		(at 54.61 36.83)
 		(diameter 0)
@@
 		(color 0 0 0 0)
 	)
+	(junction
+		(at 234.95 45.72)
+		(diameter 0)
+		(color 0 0 0 0)
+	)
 	(no_connect
 		(at 196.85 68.58)
@@
 	(wire
 		(pts
-			(xy 254 55.88) (xy 254 77.47)
-		)
-		(stroke
-			(width 0)
-			(type default)
-		)
-	)
-	(wire
-		(pts
 			(xy 97.79 34.29) (xy 97.79 36.83)
 		)
@@
 	(wire
 		(pts
+			(xy 246.38 48.26) (xy 278.13 48.26)
+		)
+		(stroke
+			(width 0)
+			(type default)
+		)
+	)
+	(wire
+		(pts
 			(xy 154.94 137.16) (xy 154.94 138.43)
 		)
@@
 	(wire
 		(pts
-			(xy 254 55.88) (xy 274.32 55.88)
+			(xy 232.41 55.88) (xy 274.32 55.88)
 		)
 		(stroke
@@
 	(wire
 		(pts
+			(xy 234.95 45.72) (xy 278.13 45.72)
+		)
+		(stroke
+			(width 0)
+			(type default)
+		)
+	)
+	(wire
+		(pts
 			(xy 195.58 76.2) (xy 196.85 76.2)
 		)
@@
 	(wire
 		(pts
-			(xy 254 85.09) (xy 254 87.63)
+			(xy 257.81 50.8) (xy 278.13 50.8)
 		)
 		(stroke
@@
 	(wire
 		(pts
-			(xy 232.41 55.88) (xy 254 55.88)
-		)
-		(stroke
-			(width 0)
-			(type default)
-		)
-	)
-	(wire
-		(pts
 			(xy 60.96 58.42) (xy 80.01 58.42)
 		)
@@
 		)
 	)
+	(hierarchical_label "U9-VDD3_1"
+		(shape output)
+		(at 278.13 50.8 0)
+		(fields_autoplaced yes)
+		(effects
+			(font
+				(size 1.27 1.27)
+			)
+			(justify left)
+		)
+	)
 	(hierarchical_label "BO"
 		(shape output)
@@
 		)
 	)
+	(hierarchical_label "U9-VDD1_1"
+		(shape output)
+		(at 278.13 45.72 0)
+		(fields_autoplaced yes)
+		(effects
+			(font
+				(size 1.27 1.27)
+			)
+			(justify left)
+		)
+	)
+	(hierarchical_label "U9-VDD2_1"
+		(shape output)
+		(at 278.13 48.26 0)
+		(fields_autoplaced yes)
+		(effects
+			(font
+				(size 1.27 1.27)
+			)
+			(justify left)
+		)
+	)
 	(symbol
 		(lib_id "power:+1V2")
@@
 	)
 	(symbol
-		(lib_id "Device:R")
-		(at 254 81.28 0)
-		(unit 1)
-		(exclude_from_sim no)
-		(in_bom yes)
-		(on_board yes)
-		(dnp no)
-		(property "Reference" "R49"
-			(at 251.714 80.772 90)
-			(effects
-				(font
-					(size 1.27 1.27)
-				)
-			)
-		)
-		(property "Value" "10k"
-			(at 255.905 80.645 90)
-			(effects
-				(font
-					(size 1.27 1.27)
-				)
-			)
-		)
-		(property "Footprint" "Resistor_SMD:R_0805_2012Metric"
-			(at 252.222 81.28 90)
-			(effects
-				(font
-					(size 1.27 1.27)
-				)
-				(hide yes)
-			)
-		)
-		(property "Datasheet" "~"
-			(at 254 81.28 0)
-			(effects
-				(font
-					(size 1.27 1.27)
-				)
-				(hide yes)
-			)
-		)
-		(property "Description" ""
-			(at 254 81.28 0)
-			(effects
-				(font
-					(size 1.27 1.27)
-				)
-				(hide yes)
-			)
-		)
-		(pin "1"
-		)
-		(pin "2"
-		)
-		(instances
-			(project "Nerd8"
-				(path "/e63e39d7-6ac0-4ffd-8aa3-1841a4541b55/4cf9c075-d009-4c35-9949-adda70ae20c7/28204049-6946-49e4-955c-4210ae323a25"
-					(reference "R49")
-					(unit 1)
-				)
-			)
-		)
-	)
-	(symbol
 		(lib_id "Device:C")
 		(at 60.96 36.83 90)
@@
 					(unit 1)
 				)
-			)
-		)
-	)
-	(symbol
-		(lib_id "power:+1V8")
-		(at 254 87.63 180)
-		(unit 1)
-		(exclude_from_sim no)
-		(in_bom yes)
-		(on_board yes)
-		(dnp no)
-		(property "Reference" "#PWR0363"
-			(at 254 83.82 0)
-			(effects
-				(font
-					(size 1.27 1.27)
-				)
-				(hide yes)
-			)
-		)
-		(property "Value" "GND"
-			(at 254 92.71 90)
-			(effects
-				(font
-					(size 1.27 1.27)
-				)
-			)
-		)
-		(property "Footprint" ""
-			(at 254 87.63 0)
-			(effects
-				(font
-					(size 1.27 1.27)
-				)
-				(hide yes)
-			)
-		)
-		(property "Datasheet" ""
-			(at 254 87.63 0)
-			(effects
-				(font
-					(size 1.27 1.27)
-				)
-				(hide yes)
-			)
-		)
-		(property "Description" ""
-			(at 254 87.63 0)
-			(effects
-				(font
-					(size 1.27 1.27)
-				)
-				(hide yes)
-			)
-		)
-		(pin "1"
-		)
-		(instances
-			(project "Nerd8"
-				(path "/e63e39d7-6ac0-4ffd-8aa3-1841a4541b55/4cf9c075-d009-4c35-9949-adda70ae20c7/28204049-6946-49e4-955c-4210ae323a25"
-					(reference "#PWR0363")
-					(unit 1)
-				)

Commit message: DRC strikes back
Connections:
- net U9-VDD1_1: now also C67.2, C69.1, U9.28 (VDD1_1); no longer C63.2, C66.1, U9.30 (VDD3_1)
- net U9-VDD3_1: now also C63.2, C66.1, U9.30 (VDD3_1); no longer C67.2, C69.1, U9.28 (VDD1_1)
Changed lines of the file:
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@@
 		)
 	)
-	(hierarchical_label "U9-VDD3_1"
+	(hierarchical_label "U9-VDD1_1"
 		(shape output)
 		(at 278.13 50.8 0)
@@
 		)
 	)
-	(hierarchical_label "U9-VDD1_1"
+	(hierarchical_label "U9-VDD3_1"
 		(shape output)
 		(at 278.13 45.72 0)
