File: bm1366.kicad_sch (KiCad schematic)
At the start: 7 parts, among them J2 Conn_01x06, U35 TXU0304PW, U8 25MHz

Commit message: DRC Check
Other:
- sheet BM1368 ports: added U9-VDD1_1, U9-VDD2_1, U9-VDD3_1; removed none
- sheet BM1368-1 ports: added U11-VDD1_1, U11-VDD2_1, U11-VDD3_1, U9-VDD1_1, U9-VDD2_1, U9-VDD3_1; removed none
- sheet BM1368-2 ports: added U11-VDD1_1, U11-VDD2_1, U11-VDD3_1, U13-VDD1_1, U13-VDD2_1, U13-VDD3_1; removed none
- sheet BM1368-3 ports: added U13-VDD1_1, U13-VDD2_1, U13-VDD3_1; removed none

Commit message: Bom
Parts:
- U8: Distributor (none) -> D; OrderNr (none) -> 1923-1664-1-ND
Changed lines of the file:
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@@
+			)
+		)
+		(property "Distributor" "D"
+			(at 49.53 85.09 0)
+			(effects
+				(font
+					(size 1.27 1.27)
+				)
+				(hide yes)
+			)
+		)
+		(property "OrderNr" "1923-1664-1-ND"
+			(at 49.53 85.09 0)
+			(effects
+				(font
+					(size 1.27 1.27)
+				)
+				(hide yes)
 			)
 		)
