File: Nerd8.kicad_sch (KiCad schematic)
At the start: 3 parts, among them J1 Conn_01x04

Commit message: Add Bom
Added iBom / DK-Bom / JLCProduction files
Parts:
- F1: OrderNr F1228CT-ND -> F2592CT-ND
Changed lines of the file:
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@@
 			)
 		)
-		(property "OrderNr" "F1228CT-ND"
+		(property "OrderNr" "F2592CT-ND"
 			(at 50.165 52.07 0)
 			(effects

Commit message: Update Nerd8.kicad_sch
Parts:
- F1: OrderNr F2592CT-ND -> F1251CT-ND
Changed lines of the file:
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@@
 			)
 		)
-		(property "OrderNr" "F2592CT-ND"
+		(property "OrderNr" "F1251CT-ND"
 			(at 50.165 52.07 0)
 			(effects
