File: power.kicad_sch (KiCad schematic)
At the start: 116 parts, among them J3 Conn_01x01, J4 Conn_01x01, U16 CSD95472Q5MC, U3 TPS53647, U36 MCP1824T-1802E, U4 CSD95472Q5MC, U5 CSD95472Q5MC, U6 AP3211, U7 MCP1824T-0802E

Commit message: Add Bom
Added iBom / DK-Bom / JLCProduction files
Parts:
- C112, C117, C181: Distributor (none) -> D; OrderNr (none) -> 490-8291-1-ND
- C3: Distributor (none) -> D; OrderNr (none) -> 478-KGM15ACG2A120JMCT-ND
- R1: Distributor (none) -> D; OrderNr (none) -> 541-16.5KCCT-ND
- R3: Distributor (none) -> D; OrderNr (none) -> 311-66.5KCRCT-ND
- R34: Distributor (none) -> D; OrderNr (none) -> RMCF0805FT16K2CT-ND
- R5: Distributor (none) -> D; OrderNr (none) -> RMCF0805FT121KCT-ND
- R7: Distributor (none) -> D; OrderNr (none) -> 311-2.55KCRCT-ND
Changed lines of the file:
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@@
 			)
 		)
-		(property "Distributor" ""
+		(property "Distributor" "D"
 			(at 62.23 154.94 0)
 			(effects
@@
 			)
 		)
-		(property "OrderNr" ""
+		(property "OrderNr" "478-KGM15ACG2A120JMCT-ND"
 			(at 62.23 154.94 0)
 			(effects
@@
 			)
 		)
+		(property "Distributor" "D"
+			(at 125.73 97.155 90)
+			(effects
+				(font
+					(size 1.27 1.27)
+				)
+				(hide yes)
+			)
+		)
+		(property "OrderNr" "541-16.5KCCT-ND"
+			(at 125.73 97.155 90)
+			(effects
+				(font
+					(size 1.27 1.27)
+				)
+				(hide yes)
+			)
+		)
 		(pin "1"
 		)
@@
 			)
 		)
-		(property "Distributor" ""
+		(property "Distributor" "D"
 			(at 303.53 26.67 0)
 			(effects
@@
 			)
 		)
-		(property "OrderNr" ""
+		(property "OrderNr" "490-8291-1-ND"
 			(at 303.53 26.67 0)
 			(effects
@@
 			)
 		)
-		(property "Distributor" ""
+		(property "Distributor" "D"
 			(at 303.53 49.53 0)
 			(effects
@@
 			)
 		)
-		(property "OrderNr" ""
+		(property "OrderNr" "490-8291-1-ND"
 			(at 303.53 49.53 0)
 			(effects
@@
 			)
 		)
-		(property "Distributor" ""
+		(property "Distributor" "D"
 			(at 173.355 212.725 0)
 			(effects
@@
 			)
 		)
-		(property "OrderNr" ""
+		(property "OrderNr" "RMCF0805FT16K2CT-ND"
 			(at 173.355 212.725 0)
 			(effects
@@
 			)
 		)
+		(property "Distributor" "D"
+			(at 40.64 119.38 90)
+			(effects
+				(font
+					(size 1.27 1.27)
+				)
+				(hide yes)
+			)
+		)
+		(property "OrderNr" "311-66.5KCRCT-ND"
+			(at 40.64 119.38 90)
+			(effects
+				(font
+					(size 1.27 1.27)
+				)
+				(hide yes)
+			)
+		)
 		(pin "1"
 		)
@@
 			)
 		)
-		(property "Distributor" ""
+		(property "Distributor" "D"
 			(at 303.53 71.755 0)
 			(effects
@@
 			)
 		)
-		(property "OrderNr" ""
+		(property "OrderNr" "490-8291-1-ND"
 			(at 303.53 71.755 0)
 			(effects
@@
 			)
 		)
+		(property "Distributor" "D"
+			(at 78.74 156.21 90)
+			(effects
+				(font
+					(size 1.27 1.27)
+				)
+				(hide yes)
+			)
+		)
+		(property "OrderNr" "311-2.55KCRCT-ND"
+			(at 78.74 156.21 90)
+			(effects
+				(font
+					(size 1.27 1.27)
+				)
+				(hide yes)
+			)
+		)
 		(pin "1"
 		)
@@
 			(effects
 				(font
+					(size 1.27 1.27)
+				)
+				(hide yes)
+			)
+		)
+		(property "Distributor" "D"
+			(at 62.23 92.71 90)
+			(effects
+				(font
+					(size 1.27 1.27)
+				)
+				(hide yes)
+			)
+		)
+		(property "OrderNr" "RMCF0805FT121KCT-ND"
+			(at 62.23 92.71 90)
+			(effects
+				(font

Commit message: Update power.kicad_sch
Parts:
- removed HS1: Heatsink, symbol Mechanical:Heatsink
Changed lines of the file:
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@@
-	)
-	(symbol
-		(lib_id "Mechanical:Heatsink")
-		(at 21.59 271.78 0)
-		(unit 1)
-		(exclude_from_sim yes)
-		(in_bom yes)
-		(on_board yes)
-		(dnp no)
-		(fields_autoplaced yes)
-		(property "Reference" "HS1"
-			(at 25.4 268.6049 0)
-			(effects
-				(font
-					(size 1.27 1.27)
-				)
-				(justify left)
-			)
-		)
-		(property "Value" "Heatsink"
-			(at 25.4 271.1449 0)
-			(effects
-				(font
-					(size 1.27 1.27)
-				)
-				(justify left)
-			)
-		)
-		(property "Footprint" ""
-			(at 21.8948 271.78 0)
-			(effects
-				(font
-					(size 1.27 1.27)
-				)
-				(hide yes)
-			)
-		)
-		(property "Datasheet" "~"
-			(at 21.8948 271.78 0)
-			(effects
-				(font
-					(size 1.27 1.27)
-				)
-				(hide yes)
-			)
-		)
-		(property "Description" "Heatsink 6.35x19.05"
-			(at 21.59 271.78 0)
-			(effects
-				(font
-					(size 1.27 1.27)
-				)
-				(hide yes)
-			)
-		)
-		(property "Distributor" "D"
-			(at 21.59 271.78 0)
-			(effects
-				(font
-					(size 1.27 1.27)
-				)
-				(hide yes)
-			)
-		)
-		(property "Manufacturer" "501100B00000G"
-			(at 21.59 271.78 0)
-			(effects
-				(font
-					(size 1.27 1.27)
-				)
-				(hide yes)
-			)
-		)
-		(property "OrderNr" "501100B00000G-ND"
-			(at 21.59 271.78 0)
-			(effects
-				(font
-					(size 1.27 1.27)
-				)
-				(hide yes)
-			)
-		)
-		(instances
-			(project "Nerd8"
-				(path "/e63e39d7-6ac0-4ffd-8aa3-1841a4541b55/8ec0a9c6-2b78-44ef-a83d-9047d2828409"
-					(reference "HS1")
-					(unit 1)
-				)
-			)
-		)
 	)
 	(symbol
